File: cc2652rb.kicad_sch (KiCad schematic)
At the start: 34 parts, among them Y1 32.768kHz, Y2 Q22FA12800150

Commit message: add POE schematics, Ethernet phy
Parts:
- added J3: JTAG, Connector:Tag-Connect_TC2030-IDC-NL_2x03_P1.27mm_Vertical, symbol Connector:Conn_ARM_SWD_TagConnect_TC2030-NL
- renumbered L to L4, L to L5, L to L6, L to L7
Connections:
- net GND: now also J3.5 (GND)
- net JTAG_TCK: now also J3.4 (SWCLK)
- net JTAG_TDI: now also J3.2 (SWDIO)
- net JTAG_TDO: now also J3.6 (SWO)
- net JTAG_TMS: now also J3.1 (VCC)
- net nRESET: now also J3.3 (~{RESET})
Changed lines of the file:
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@@
   (no_connect (at 151.13 95.25))
   (no_connect (at 151.13 100.33))
+  (wire (pts (xy 260.35 121.92) (xy 262.89 121.92))
+    (stroke (width 0) (type default))
+  )
   (wire (pts (xy 71.12 85.09) (xy 74.93 85.09))
     (stroke (width 0) (type default))
@@
     (stroke (width 0) (type default))
   )
+  (wire (pts (xy 260.35 116.84) (xy 262.89 116.84))
+    (stroke (width 0) (type default))
+  )
   (wire (pts (xy 151.13 113.03) (xy 123.19 113.03))
     (stroke (width 0) (type default))
@@
     (stroke (width 0) (type default))
   )
+  (wire (pts (xy 260.35 111.76) (xy 262.89 111.76))
+    (stroke (width 0) (type default))
+  )
   (wire (pts (xy 71.12 113.03) (xy 74.93 113.03))
     (stroke (width 0) (type default))
@@
     (stroke (width 0) (type default))
   )
+  (wire (pts (xy 260.35 119.38) (xy 262.89 119.38))
+    (stroke (width 0) (type default))
+  )
   (wire (pts (xy 78.74 35.56) (xy 76.2 35.56))
     (stroke (width 0) (type default))
@@
     )
   )
+  (global_label "nRESET" (shape input) (at 260.35 111.76 180) (fields_autoplaced)
+    (effects (font (size 1.27 1.27)) (justify right))
+    (property "Intersheetrefs" "${INTERSHEET_REFS}" (at 250.4707 111.76 0)
+      (effects (font (size 1.27 1.27)) (justify right) hide)
+    )
+  )
   (global_label "X32Q1" (shape input) (at 48.26 113.03 180) (fields_autoplaced)
     (effects (font (size 1.27 1.27)) (justify right))
@@
     )
   )
+  (global_label "JTAG_TDO" (shape input) (at 260.35 121.92 180) (fields_autoplaced)
+    (effects (font (size 1.27 1.27)) (justify right))
+    (property "Intersheetrefs" "${INTERSHEET_REFS}" (at 248.5353 121.92 0)
+      (effects (font (size 1.27 1.27)) (justify right) hide)
+    )
+  )
+  (global_label "JTAG_TMS" (shape input) (at 273.05 106.68 90) (fields_autoplaced)
+    (effects (font (size 1.27 1.27)) (justify left))
+    (property "Intersheetrefs" "${INTERSHEET_REFS}" (at 273.05 94.8049 90)
+      (effects (font (size 1.27 1.27)) (justify left) hide)
+    )
+  )
+  (global_label "JTAG_TDI" (shape input) (at 260.35 119.38 180) (fields_autoplaced)
+    (effects (font (size 1.27 1.27)) (justify right))
+    (property "Intersheetrefs" "${INTERSHEET_REFS}" (at 249.261 119.38 0)
+      (effects (font (size 1.27 1.27)) (justify right) hide)
+    )
+  )
+  (global_label "JTAG_TCK" (shape input) (at 260.35 116.84 180) (fields_autoplaced)
+    (effects (font (size 1.27 1.27)) (justify right))
+    (property "Intersheetrefs" "${INTERSHEET_REFS}" (at 248.5958 116.84 0)
+      (effects (font (size 1.27 1.27)) (justify right) hide)
+    )
+  )
   (symbol (lib_id "RF_ZigBee:CC2652RB1FRGZR") (at 153.67 48.26 0) (unit 1)
     (in_bom yes) (on_board yes) (dnp no) (fields_autoplaced)
@@
     )
   )
+  (symbol (lib_id "Connector:Conn_ARM_SWD_TagConnect_TC2030-NL") (at 270.51 116.84 0) (mirror y) (unit 1)
+    (in_bom no) (on_board yes) (dnp no) (fields_autoplaced)
+    (property "Reference" "J3" (at 276.86 115.57 0)
+      (effects (font (size 1.27 1.27)) (justify right))
+    )
+    (property "Value" "JTAG" (at 276.86 118.11 0)
+      (effects (font (size 1.27 1.27)) (justify right))
+    )
+    (property "Footprint" "Connector:Tag-Connect_TC2030-IDC-NL_2x03_P1.27mm_Vertical" (at 270.51 134.62 0)
+      (effects (font (size 1.27 1.27)) hide)
+    )
+    (property "Datasheet" "https://www.tag-connect.com/wp-content/uploads/bsk-pdf-manager/TC2030-CTX_1.pdf" (at 270.51 132.08 0)
+      (effects (font (size 1.27 1.27)) hide)
+    )
+    (pin "1")
+    (pin "2")
+    (pin "3")
+    (pin "4")
+    (pin "5")
+    (pin "6")
+    (instances
+      (project "stm32f745-eth-can-sdram"
+        (path "/2fe210a3-bd39-4a0d-882e-a71d33b1f0de/6d2ec507-6229-4b8e-90ca-829229a57347"
+          (reference "J3") (unit 1)
+        )
+      )
+    )
+  )
   (symbol (lib_id "Device:C") (at 52.07 116.84 0) (unit 1)
     (in_bom yes) (on_board yes) (dnp no) (fields_autoplaced)
@@
   (symbol (lib_id "Device:LQG15HS") (at 134.62 39.37 90) (unit 1)
     (in_bom yes) (on_board yes) (dnp no)
-    (property "Reference" "L" (at 132.08 39.37 0)
+    (property "Reference" "L7" (at 132.08 39.37 0)
       (effects (font (size 1.27 1.27)))
     )
@@
       (project "stm32f745-eth-can-sdram"
         (path "/2fe210a3-bd39-4a0d-882e-a71d33b1f0de/6d2ec507-6229-4b8e-90ca-829229a57347"
-          (reference "L") (unit 1)
+          (reference "L7") (unit 1)
         )
       )
@@
   (symbol (lib_id "Device:LQG15HS") (at 83.82 50.8 0) (mirror y) (unit 1)
     (in_bom yes) (on_board yes) (dnp no)
-    (property "Reference" "L" (at 83.82 48.26 0)
+    (property "Reference" "L4" (at 83.82 48.26 0)
       (effects (font (size 1.27 1.27)))
     )
@@
       (project "stm32f745-eth-can-sdram"
         (path "/2fe210a3-bd39-4a0d-882e-a71d33b1f0de/6d2ec507-6229-4b8e-90ca-829229a57347"
-          (reference "L") (unit 1)
+          (reference "L4") (unit 1)
         )
       )
@@
     )
   )
+  (symbol (lib_id "power:GND") (at 273.05 127 0) (unit 1)
+    (in_bom yes) (on_board yes) (dnp no) (fields_autoplaced)
+    (property "Reference" "#PWR070" (at 273.05 133.35 0)
+      (effects (font (size 1.27 1.27)) hide)
+    )
+    (property "Value" "GND" (at 273.05 132.08 0)
+      (effects (font (size 1.27 1.27)))
+    )
+    (property "Footprint" "" (at 273.05 127 0)
+      (effects (font (size 1.27 1.27)) hide)
+    )
+    (property "Datasheet" "" (at 273.05 127 0)
+      (effects (font (size 1.27 1.27)) hide)
+    )
+    (pin "1")
+    (instances
+      (project "stm32f745-eth-can-sdram"
+        (path "/2fe210a3-bd39-4a0d-882e-a71d33b1f0de/6d2ec507-6229-4b8e-90ca-829229a57347"
+          (reference "#PWR070") (unit 1)
+        )
+      )
+    )
+  )
   (symbol (lib_id "Device:C") (at 101.6 154.94 0) (unit 1)
     (in_bom yes) (on_board yes) (dnp no) (fields_autoplaced)
@@
   (symbol (lib_id "Device:LQG15HS") (at 125.73 55.88 0) (mirror y) (unit 1)
     (in_bom yes) (on_board yes) (dnp no)
-    (property "Reference" "L" (at 125.73 53.34 0)
+    (property "Reference" "L6" (at 125.73 53.34 0)
       (effects (font (size 1.27 1.27)))
     )
@@
       (project "stm32f745-eth-can-sdram"
         (path "/2fe210a3-bd39-4a0d-882e-a71d33b1f0de/6d2ec507-6229-4b8e-90ca-829229a57347"
-          (reference "L") (unit 1)
+          (reference "L6") (unit 1)
         )
       )
@@
   (symbol (lib_id "Device:LQG15HS") (at 104.14 50.8 0) (mirror y) (unit 1)
     (in_bom yes) (on_board yes) (dnp no)
-    (property "Reference" "L" (at 104.14 48.26 0)
+    (property "Reference" "L5" (at 104.14 48.26 0)
       (effects (font (size 1.27 1.27)))
     )
@@
       (project "stm32f745-eth-can-sdram"
         (path "/2fe210a3-bd39-4a0d-882e-a71d33b1f0de/6d2ec507-6229-4b8e-90ca-829229a57347"
-          (reference "L") (unit 1)
+          (reference "L5") (unit 1)
         )
       )

Commit message: almost final schematics
Parts:
- removed C4 (x2): 1pF, Capacitor_SMD:C_0402_1005Metric, symbol Device:C
- added C4 (x2): 12pF, Capacitor_SMD:C_0402_1005Metric, symbol Device:C
- J2: footprint (none) -> RF_Antenna:SMA_RF_SMD
- R1: footprint (none) -> Resistor_SMD:R_0402_1005Metric
Connections:
- net GND: now also J2.1, C4.2, C4.2; no longer J2.3, J2.4, J2.5
- net X32Q1: now also C4.1
- net X32Q2: now also C4.1
- net at C4.1: now also J2.3; no longer J2.1
Other:
- note removed: "do not place"
- moved on the sheet: C4
