File: sdram.kicad_sch (KiCad schematic)
At the start: 0 parts

Commit message: almost final schematics
Parts:
- added C4 (x14): 100n, Capacitor_SMD:C_0402_1005Metric, symbol Device:C
- added R1 (x18): 10K, Resistor_SMD:R_0402_1005Metric, symbol Device:R
- added U11: IS42S32800J-7BLI, Package_BGA:BGA-90_8.0x13.0mm_Layout2x3x15_P0.8mm, symbol Memory_RAM:IS42S32800J-7BLI
Connections:
- new net: R1.1, U11.C2 (DQ27)
- new net: R1.1, U11.D8 (DQ18)
- new net: R1.1, U11.B9 (DQ19)
- new net: R1.1, U11.B1 (DQ28)
- new net: R1.1, U11.C3 (DQ25)
- new net: R1.1, U11.E2 (DQ31)
- new net: R1.1, U11.D3 (DQ30)
- new net: R1.1, U11.E8 (DQ16)
- new net: R1.1, U11.A1 (DQ26)
- new net: R1.1, U11.A9 (DQ21)
- new net: R1.1, U11.F8 (DQM2)
- new net: R1.1, U11.A2 (DQ24)
- new net: R1.1, U11.A8 (DQ23)
- new net: R1.1, U11.C7 (DQ22)
- new net: R1.1, U11.C8 (DQ20)
- new net: R1.1, U11.D2 (DQ29)
- new net: R1.1, U11.D7 (DQ17)
- new net: R1.1, U11.F2 (DQM3)
- new net +3.3V: C4.1, C4.1, C4.1, C4.1, C4.1, C4.1, C4.1, C4.1, C4.1, C4.1, C4.1, C4.1, C4.1, C4.1, U11.A7 (VDD), U11.B2 (VDDQ), U11.B7 (VDDQ), U11.C9 (VDDQ), U11.D9 (VDDQ), U11.E1 (VDDQ), U11.F9 (VDD), U11.L1 (VDDQ), U11.L7 (VDD), U11.M9 (VDDQ), U11.N9 (VDDQ), U11.P2 (VDDQ), U11.P7 (VDDQ), U11.R7 (VDD)
- new net FMC_A0: U11.G8 (A0)
- new net FMC_A1: U11.G9 (A1)
- new net FMC_A10: U11.G7 (A10)
- new net FMC_A11: U11.H9 (A11)
- new net FMC_A2: U11.F7 (A2)
- new net FMC_A3: U11.F3 (A3)
- new net FMC_A4: U11.G1 (A4)
- new net FMC_A5: U11.G2 (A5)
- new net FMC_A6: U11.G3 (A6)
- new net FMC_A7: U11.H1 (A7)
- new net FMC_A8: U11.H2 (A8)
- new net FMC_A9: U11.J3 (A9)
- new net FMC_BA0: U11.J7 (BA0)
- new net FMC_BA1: U11.H8 (BA1)
- new net FMC_D0: U11.R8 (DQ0)
- new net FMC_D1: U11.N7 (DQ1)
- new net FMC_D10: U11.M2 (DQ10)
- new net FMC_D11: U11.P1 (DQ11)
- new net FMC_D12: U11.N2 (DQ12)
- new net FMC_D13: U11.R1 (DQ13)
- new net FMC_D14: U11.N3 (DQ14)
- new net FMC_D15: U11.R2 (DQ15)
- new net FMC_D2: U11.R9 (DQ2)
- new net FMC_D3: U11.N8 (DQ3)
- new net FMC_D4: U11.P9 (DQ4)
- new net FMC_D5: U11.M8 (DQ5)
- new net FMC_D6: U11.M7 (DQ6)
- new net FMC_D7: U11.L8 (DQ7)
- new net FMC_D8: U11.L2 (DQ8)
- new net FMC_D9: U11.M3 (DQ9)
- new net FMC_NBL0: U11.K9 (DQM0)
- new net FMC_NBL1: U11.K1 (DQM1)
- new net FMC_SDCKE0: U11.J2 (CKE)
- new net FMC_SDCLK: U11.J1 (CLK)
- new net FMC_SDNCAS: U11.K7 (~{CAS})
- new net FMC_SDNE0: U11.J8 (~{CS})
- new net FMC_SDNRAS: U11.J9 (~{RAS})
- new net FMC_SDNWE: U11.K8 (~{WE})
- new net GND: C4.2, C4.2, C4.2, C4.2, C4.2, C4.2, C4.2, C4.2, C4.2, C4.2, C4.2, C4.2, C4.2, C4.2, R1.2, R1.2, R1.2, R1.2, R1.2, R1.2, R1.2, R1.2, R1.2, R1.2, R1.2, R1.2, R1.2, R1.2, R1.2, R1.2, R1.2, R1.2, U11.A3 (VSS), U11.B3 (VSSQ), U11.B8 (VSSQ), U11.C1 (VSSQ), U11.D1 (VSSQ), U11.E9 (VSSQ), U11.F1 (VSS), U11.L3 (VSS), U11.L9 (VSSQ), U11.M1 (VSSQ), U11.N1 (VSSQ), U11.P3 (VSSQ), U11.P8 (VSSQ), U11.R3 (VSS)
- no-connect marks 0 -> 6
